Commit message: added readme

File: husky_bot/description/urdf/decorations.urdf.xacro (robot description, xacro)
@@ -33,4 +33,7 @@
       </visual>
     </link>
+    <gazebo reference="top_chassis_link">
+      <material>Gazebo/Orange</material>
+      </gazebo>
     <!-- Attach chassis to the robot -->
     <joint name="top_chassis_joint" type="fixed">
@@ -62,4 +65,7 @@
       </visual>
     </link>
+    <gazebo reference="front_bumper_link">
+    <material>Gazebo/Green</material>
+    </gazebo>
     <!-- Attach front bumper -->
     <joint name="front_bumper" type="fixed">
@@ -181,4 +187,7 @@
       <link name="top_plate_rear_link"/>
     </xacro:if>
+         <gazebo reference="top_plate_link">
+      <material>Gazebo/Green</material>
+      </gazebo>
   </xacro:macro>
 </robot>

File: husky_bot/description/urdf/husky.urdf.xacro (robot description, xacro)
@@ -37,4 +37,6 @@
   <xacro:include filename="$(find husky_bot)/description/urdf/accessories/sick_lms1xx_mount.urdf.xacro"/>
   <xacro:include filename="$(find husky_bot)/description/urdf/accessories/sensor_arch.urdf.xacro"/>
+   <!-- Import Rviz colors -->
+  <xacro:include filename="$(find husky_bot)/description/urdf/materials.xacro" />
   <xacro:property name="M_PI" value="3.14159"/>
   <!-- Base Size -->
@@ -49,15 +51,4 @@
   <xacro:property name="wheel_length" value="0.1143" />
   <xacro:property name="wheel_radius" value="0.1651" />
-  <!-- materials -->
-  <xacro:property name="material_white">
-    <material name="white">
-      <color rgba="1 1 1 1"/>
-    </material>
-  </xacro:property>
-  <xacro:property name="material_orange">
-    <material name="orange">
-      <color rgba="1.0 0.7 0.0 1"/>
-    </material>
-  </xacro:property>
   <!-- Base link is the center of the robot's bottom plate -->
   <link name="base_link">
@@ -67,4 +58,5 @@
         <mesh filename="package://husky_bot/description/meshes/base_link.dae" />
       </geometry>
+      <material name="green"/>
     </visual>
     <collision>
@@ -125,4 +117,10 @@
   </xacro:husky_wheel>
   <xacro:husky_decorate />
+  <gazebo reference="base_link">
+  <material>Gazebo/Orange</material>
+  </gazebo>
+   <gazebo reference="imu_link">
+  <material>Gazebo/Green</material>
+  </gazebo>
   <xacro:if value="$(arg laser_enabled)">
     <sick_lms1xx_mount prefix="base"/>

File: husky_bot/description/urdf/wheel.urdf.xacro (robot description, xacro)
@@ -49,5 +49,5 @@
 			<kd value="1.0" />
 			<fdir1 value="1 0 0"/>
-			<material name="orange"/>
+			<material>Gazebo/White</material>
 		</gazebo>
 		<joint name="${wheel_prefix}_wheel" type="continuous">
